Commit message: added up to date URDF files for the robot

File: src/robot_description/urdf/qbert.urdf (robot description, URDF)
Before this commit: robot qbert, 1 links, 0 joints
Links:
- added link Origin, mass 1e-9
- added link axe, mass 1e-9
- added link camera_left, mass 1e-9
- added link camera_right, mass 1e-9
- added link compressor, mass 0.601925; collision mesh filename=package://meshes/merged/compressor_collision.stl; visual mesh filename=package://meshes/merged/compressor_visual.stl
- added link compressor_2, mass 0.601925; collision mesh filename=package://meshes/merged/compressor_2_collision.stl; visual mesh filename=package://meshes/merged/compressor_2_visual.stl
- added link compressor_3, mass 0.601925; collision mesh filename=package://meshes/merged/compressor_3_collision.stl; visual mesh filename=package://meshes/merged/compressor_3_visual.stl
- added link compressor_4, mass 0.601925; collision mesh filename=package://meshes/merged/compressor_4_collision.stl; visual mesh filename=package://meshes/merged/compressor_4_visual.stl
- added link roller_gripper, mass 0.549326; collision mesh filename=package://meshes/merged/roller_gripper_collision.stl; visual mesh filename=package://meshes/merged/roller_gripper_visual.stl
- added link roller_gripper_2, mass 0.549326; collision mesh filename=package://meshes/merged/roller_gripper_2_collision.stl; visual mesh filename=package://meshes/merged/roller_gripper_2_visual.stl
- added link roller_gripper_3, mass 0.549326; collision mesh filename=package://meshes/merged/roller_gripper_3_collision.stl; visual mesh filename=package://meshes/merged/roller_gripper_3_visual.stl
- added link roller_gripper_4, mass 0.549326; collision mesh filename=package://meshes/merged/roller_gripper_4_collision.stl; visual mesh filename=package://meshes/merged/roller_gripper_4_visual.stl
- added link rot_disc, mass 10.8297; collision mesh filename=package://meshes/merged/rot_disc_collision.stl; visual mesh filename=package://meshes/merged/rot_disc_visual.stl
- added link solid_gripper, mass 0.940003; collision mesh filename=package://meshes/merged/solid_gripper_collision.stl; visual mesh filename=package://meshes/merged/solid_gripper_visual.stl
- added link solid_gripper_2, mass 0.940003; collision mesh filename=package://meshes/merged/solid_gripper_2_collision.stl; visual mesh filename=package://meshes/merged/solid_gripper_2_visual.stl
- added link solid_gripper_3, mass 0.940003; collision mesh filename=package://meshes/merged/solid_gripper_3_collision.stl; visual mesh filename=package://meshes/merged/solid_gripper_3_visual.stl
- added link solid_gripper_4, mass 0.940003; collision mesh filename=package://meshes/merged/solid_gripper_4_collision.stl; visual mesh filename=package://meshes/merged/solid_gripper_4_visual.stl
- added link stator, mass 4.59951; collision mesh filename=package://meshes/merged/stator_collision.stl; visual mesh filename=package://meshes/merged/stator_visual.stl
- added link tooling_disc, mass 7.26529; collision mesh filename=package://meshes/merged/tooling_disc_collision.stl; visual mesh filename=package://meshes/merged/tooling_disc_visual.stl
- added link unstrander, mass 1e-9
- added link unstrander_2, mass 0.0687236; collision mesh filename=package://meshes/merged/unstrander_2_collision.stl; visual mesh filename=package://meshes/merged/unstrander_2_visual.stl
- link linear_gantry__configuration_festo: mass 1.22887 -> 0.374514; geometry collision mesh filename=package://meshes/merged/linear_gantry__configuration_festo_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; visual mesh filename=package://meshes/merged/linear_gantry__configuration_festo_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
Joints:
- added joint J1_gantry: type prismatic, parent linear_gantry__configuration_festo, child stator, origin xyz=-0.285903 -0.0647361 0.174215 rpy=1.5708 -1.5708 0, axis 0 0 1, limit lower=-0.27 upper=0.27 effort=10 velocity=10
- added joint J2_A_rotor: type revolute, parent stator, child rot_disc, origin xyz=0.27825 -0.14 0.2 rpy=-3.14159 2.69849e-15 -1.57513, axis 0 0 1, limit lower=-3.14593 upper=3.13726 effort=10 velocity=10
- added joint J2_B_solid_gripper_1: type prismatic, parent stator, child solid_gripper, origin xyz=0.10415 -0.14 -0.153 rpy=-1.5708 7.21582e-15 1.5708, axis 0 0 1, limit lower=-0.04 upper=0 effort=10 velocity=10
- added joint J2_B_solid_gripper_2: type prismatic, parent stator, child solid_gripper_2, origin xyz=0.27825 -0.3141 -0.153 rpy=-1.5708 2.27583e-14 -3.14159, axis 0 0 1, limit lower=-0.04 upper=-6.38378e-16 effort=10 velocity=10, mimic joint=J2_B_solid_gripper_1 multiplier=1.0
- added joint J2_B_solid_gripper_3: type prismatic, parent stator, child solid_gripper_3, origin xyz=0.27825 0.0341 -0.153 rpy=1.5708 -4.08537e-14 -3.14159, axis 0 0 1, limit lower=-0.04 upper=-3.88578e-16 effort=10 velocity=10, mimic joint=J2_B_solid_gripper_1 multiplier=1.0
- added joint J2_B_solid_gripper_4: type prismatic, parent stator, child solid_gripper_4, origin xyz=0.45235 -0.14 -0.153 rpy=1.5708 -4.82829e-14 1.5708, axis 0 0 1, limit lower=-0.04 upper=-4.44089e-16 effort=10 velocity=10, mimic joint=J2_B_solid_gripper_1 multiplier=1.0
- added joint J2_C_roller_gripper_1: type prismatic, parent stator, child roller_gripper, origin xyz=0.131101 0.00714892 -0.229 rpy=1.5708 8.34931e-15 -2.35619, axis 0 0 1, limit lower=-0.04 upper=1.15402e-14 effort=10 velocity=10
- added joint J2_C_roller_gripper_2: type prismatic, parent stator, child roller_gripper_2, origin xyz=0.131101 -0.287149 -0.229 rpy=1.5708 8.75838e-16 -0.785398, axis 0 0 1, limit lower=-0.04 upper=1.15426e-14 effort=10 velocity=10, mimic joint=J2_C_roller_gripper_1 multiplier=1.0
- added joint J2_C_roller_gripper_3: type prismatic, parent stator, child roller_gripper_3, origin xyz=0.425399 -0.287149 -0.229 rpy=-1.5708 8.38912e-15 -2.35619, axis 0 0 1, limit lower=-0.04 upper=1.16236e-14 effort=10 velocity=10, mimic joint=J2_C_roller_gripper_1 multiplier=1.0
- added joint J2_C_roller_gripper_4: type prismatic, parent stator, child roller_gripper_4, origin xyz=0.425399 0.00714892 -0.229 rpy=-1.5708 6.60057e-16 -0.785398, axis 0 0 1, limit lower=-0.04 upper=1.14617e-14 effort=10 velocity=10, mimic joint=J2_C_roller_gripper_1 multiplier=1.0
- added joint J3_B_compressor_1: type prismatic, parent rot_disc, child compressor, origin xyz=3.88578e-16 -0.1911 0.081 rpy=1.5708 -4.34328e-14 -1.84623e-15, axis 0 0 1, limit lower=-0.04 upper=0.0 effort=10 velocity=10
- added joint J3_B_compressor_2: type prismatic, parent rot_disc, child compressor_2, origin xyz=0.1911 4.996e-16 0.037 rpy=1.5708 -3.30585e-15 1.5708, axis 0 0 1, limit lower=-0.04 upper=0.0 effort=10 velocity=10
- added joint J3_B_compressor_3: type prismatic, parent rot_disc, child compressor_3, origin xyz=-0.1911 -1.55431e-15 0.037 rpy=-1.5708 6.20095e-15 1.5708, axis 0 0 1, limit lower=-0.04 upper=0 effort=10 velocity=10, mimic joint=J3_B_compressor_2 multiplier=1.0
- added joint J3_B_compressor_4: type prismatic, parent rot_disc, child compressor_4, origin xyz=3.88578e-16 0.1911 0.081 rpy=-1.5708 -3.56609e-14 6.32771e-15, axis 0 0 1, limit lower=-0.04 upper=0.0 effort=10 velocity=10, mimic joint=J3_B_compressor_1 multiplier=1.0
- added joint J4_unstrander: type prismatic, parent tooling_disc, child unstrander_2, origin xyz=-0.131984 -0.231215 -0.298562 rpy=-1.5708 4.06796e-16 2.35619, axis 0 0 1, limit lower=-0.04 upper=0.0 effort=10 velocity=10
- added joint Origin_frame: type fixed, parent linear_gantry__configuration_festo, child Origin, origin xyz=-0.145903 0.362264 0.452465 rpy=-1.5708 -0 0, axis 0 0 0
- added joint axe_frame: type fixed, parent tooling_disc, child axe, origin xyz=-1.02696e-15 -0.17475 -0.323467 rpy=4.59948e-16 8.65217e-16 -1.5708, axis 0 0 0
- added joint camera_left_frame: type fixed, parent rot_disc, child camera_left, origin xyz=0.0175 -0.24505 -0.0825 rpy=-1.5708 -7.38925e-20 1.68627e-16, axis 0 0 0
- added joint camera_right_frame: type fixed, parent rot_disc, child camera_right, origin xyz=-0.0325 -0.24505 -0.0825 rpy=-1.5708 -7.38925e-20 1.68627e-16, axis 0 0 0
- added joint joint_J3_A_tool_disc: type prismatic, parent rot_disc, child tooling_disc, origin xyz=0.123567 0.123567 0.1805 rpy=1.25607e-15 -1.12739e-23 -0.785398, axis 0 0 1, limit lower=-0.2 upper=0 effort=10 velocity=10
- added joint unstrander_frame: type fixed, parent unstrander_2, child unstrander, origin xyz=-0.0534015 -0.0232676 -0.0560611 rpy=1.5708 -1.5708 0, axis 0 0 0

Commit message: made the rviz kindof work

File: src/robot_description/urdf/qbert.urdf (robot description, URDF)
Before this commit: robot qbert, 22 links, 21 joints
Links:
- link compressor: geometry collision mesh filename=package://robot_description/meshes/merged/compressor_collis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; visual mesh filename=package://robot_description/meshes/merged/compressor_visual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
- link compressor_2: geometry collision mesh filename=package://robot_description/meshes/merged/compressor_2_coll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; visual mesh filename=package://robot_description/meshes/merged/compressor_2_visu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
- link compressor_3: geometry collision mesh filename=package://robot_description/meshes/merged/compressor_3_coll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; visual mesh filename=package://robot_description/meshes/merged/compressor_3_visu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
- link compressor_4: geometry collision mesh filename=package://robot_description/meshes/merged/compressor_4_coll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; visual mesh filename=package://robot_description/meshes/merged/compressor_4_visu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
- link linear_gantry__configuration_festo: geometry collision mesh filename=package://robot_description/meshes/merged/linear_gantry__co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; visual mesh filename=package://robot_description/meshes/merged/linear_gantry__co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
- link roller_gripper: geometry collision mesh filename=package://robot_description/meshes/merged/roller_gripper_co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; visual mesh filename=package://robot_description/meshes/merged/roller_gripper_vi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
- link roller_gripper_2: geometry collision mesh filename=package://robot_description/meshes/merged/roller_gripper_2_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; visual mesh filename=package://robot_description/meshes/merged/roller_gripper_2_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
- link roller_gripper_3: geometry collision mesh filename=package://robot_description/meshes/merged/roller_gripper_3_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; visual mesh filename=package://robot_description/meshes/merged/roller_gripper_3_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
- link roller_gripper_4: geometry collision mesh filename=package://robot_description/meshes/merged/roller_gripper_4_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; visual mesh filename=package://robot_description/meshes/merged/roller_gripper_4_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
- link rot_disc: geometry collision mesh filename=package://robot_description/meshes/merged/rot_disc_collisio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; visual mesh filename=package://robot_description/meshes/merged/rot_disc_visual.s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
- link solid_gripper: geometry collision mesh filename=package://robot_description/meshes/merged/solid_gripper_col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; visual mesh filename=package://robot_description/meshes/merged/solid_gripper_vis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
- link solid_gripper_2: geometry collision mesh filename=package://robot_description/meshes/merged/solid_gripper_2_c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; visual mesh filename=package://robot_description/meshes/merged/solid_gripper_2_v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
- link solid_gripper_3: geometry collision mesh filename=package://robot_description/meshes/merged/solid_gripper_3_c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; visual mesh filename=package://robot_description/meshes/merged/solid_gripper_3_v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
- link solid_gripper_4: geometry collision mesh filename=package://robot_description/meshes/merged/solid_gripper_4_c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; visual mesh filename=package://robot_description/meshes/merged/solid_gripper_4_v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
- link stator: geometry collision mesh filename=package://robot_description/meshes/merged/stator_collision.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; visual mesh filename=package://robot_description/meshes/merged/stator_visual.stl
- link tooling_disc: geometry collision mesh filename=package://robot_description/meshes/merged/tooling_disc_coll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; visual mesh filename=package://robot_description/meshes/merged/tooling_disc_visu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
- link unstrander_2: geometry collision mesh filename=package://robot_description/meshes/merged/unstrander_2_coll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; visual mesh filename=package://robot_description/meshes/merged/unstrander_2_visu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
Joints:
- joint Origin_frame: child Origin -> linear_gantry__configuration_festo; parent linear_gantry__configuration_festo -> Origin

Commit message: working rviz setup

File: src/robot_description/urdf/qbert.urdf (robot description, URDF)
Before this commit: robot qbert, 22 links, 21 joints
Links:
- link Origin: mass 1e-9 -> None
