Commit message: fixed small issue

File: src/qbert_description/urdf/qbert.xacro (robot description, xacro)
@@ -1,5 +1,9 @@
 <?xml version="1.0"?>
 <robot xmlns:xacro="http://www.ros.org/wiki/xacro" name="qbert">
-    <xacro:include filename="$(find robot_description)/urdf/qbert_base.xacro"/>
+    <!-- Load the base model -->
+    <xacro:include filename="$(find qbert_description)/urdf/qbert_base.xacro"/>
+    <!-- Load the ros 2 control parameters -->
+    <xacro:include filename="$(find qbert_description)/urdf/qbert_ros2control.xacro"/>
+    <!-- Load gazebo plugin -->
     <gazebo>
         <plugin
@@ -19,10 +23,10 @@
     <gazebo reference="camera_left">
         <sensor name="camera" type="camera">
-            <pose> 0 0 0 0 0 0 </pose>
+            <pose> 0 0 0 -${pi/2} -${pi/2} 0 </pose>
             <visualize>true</visualize>
-            <update_rate>1</update_rate>
+            <update_rate>30</update_rate>
             <camera>
                 <camera_info_topic>camera/camera_info</camera_info_topic>
-                <horizontal_fov>1.089</horizontal_fov>
+                <horizontal_fov>${pi/2}</horizontal_fov>
                 <image>
                     <format>R8G8B8</format>
@@ -38,3 +42,9 @@
         </sensor>
     </gazebo>
+    <gazebo>
+        <plugin filename="libgz_ros2_control-system.so" name="gz_ros2_control::GazeboSimROS2ControlPlugin">
+            <parameters>$(find qbert_description)/config/qbert_controllers.yaml</parameters>
+            <controller_manager_prefix_node_name>controller_manager</controller_manager_prefix_node_name>
+        </plugin>
+    </gazebo>
 </robot>

File: src/qbert_description/urdf/qbert_base.xacro (robot description, xacro)
@@ -24,5 +24,5 @@
       <origin xyz="-0.145903 -0.0648003 0.0860613" rpy="0 -0 0"/>
       <geometry>
-        <mesh filename="package://robot_description/meshes/merged/linear_gantry__configuration_festo_visual.stl"/>
+        <mesh filename="package://qbert_description/meshes/merged/linear_gantry__configuration_festo_visual.stl"/>
       </geometry>
       <material name="linear_gantry__configuration_festo_parts_material">
@@ -33,5 +33,5 @@
       <origin xyz="-0.145903 -0.0648003 0.0860613" rpy="0 -0 0"/>
       <geometry>
-        <mesh filename="package://robot_description/meshes/merged/linear_gantry__configuration_festo_collision.stl"/>
+        <mesh filename="package://qbert_description/meshes/merged/linear_gantry__configuration_festo_collision.stl"/>
       </geometry>
     </collision>
@@ -48,5 +48,5 @@
       <origin xyz="0.27825 -0.14 -0.188372" rpy="-1.5708 -3.6585e-14 -1.5708"/>
       <geometry>
-        <mesh filename="package://robot_description/meshes/merged/stator_visual.stl"/>
+        <mesh filename="package://qbert_description/meshes/merged/stator_visual.stl"/>
       </geometry>
       <material name="stator_parts_material">
@@ -57,5 +57,5 @@
       <origin xyz="0.27825 -0.14 -0.188372" rpy="-1.5708 -3.6585e-14 -1.5708"/>
       <geometry>
-        <mesh filename="package://robot_description/meshes/merged/stator_collision.stl"/>
+        <mesh filename="package://qbert_description/meshes/merged/stator_collision.stl"/>
       </geometry>
     </collision>
@@ -72,5 +72,5 @@
       <origin xyz="4.44089e-16 5.55112e-16 0.0433903" rpy="1.5708 3.92647e-14 -0.00433337"/>
       <geometry>
-        <mesh filename="package://robot_description/meshes/merged/rot_disc_visual.stl"/>
+        <mesh filename="package://qbert_description/meshes/merged/rot_disc_visual.stl"/>
       </geometry>
       <material name="rot_disc_parts_material">
@@ -81,5 +81,5 @@
       <origin xyz="4.44089e-16 5.55112e-16 0.0433903" rpy="1.5708 3.92647e-14 -0.00433337"/>
       <geometry>
-        <mesh filename="package://robot_description/meshes/merged/rot_disc_collision.stl"/>
+        <mesh filename="package://qbert_description/meshes/merged/rot_disc_collision.stl"/>
       </geometry>
     </collision>
@@ -126,5 +126,5 @@
       <origin xyz="-0.00632037 -0.180912 -0.251556" rpy="1.5708 4.0149e-14 0.781065"/>
       <geometry>
-        <mesh filename="package://robot_description/meshes/merged/tooling_disc_visual.stl"/>
+        <mesh filename="package://qbert_description/meshes/merged/tooling_disc_visual.stl"/>
       </geometry>
       <material name="tooling_disc_parts_material">
@@ -135,5 +135,5 @@
       <origin xyz="-0.00632037 -0.180912 -0.251556" rpy="1.5708 4.0149e-14 0.781065"/>
       <geometry>
-        <mesh filename="package://robot_description/meshes/merged/tooling_disc_collision.stl"/>
+        <mesh filename="package://qbert_description/meshes/merged/tooling_disc_collision.stl"/>
       </geometry>
     </collision>
@@ -165,5 +165,5 @@
       <origin xyz="-0.0534015 -0.00511464 -0.0611991" rpy="-7.90508e-12 1.56646 3.14159"/>
       <geometry>
-        <mesh filename="package://robot_description/meshes/merged/unstrander_2_visual.stl"/>
+        <mesh filename="package://qbert_description/meshes/merged/unstrander_2_visual.stl"/>
       </geometry>
       <material name="unstrander_2_parts_material">
@@ -174,5 +174,5 @@
       <origin xyz="-0.0534015 -0.00511464 -0.0611991" rpy="-7.90508e-12 1.56646 3.14159"/>
       <geometry>
-        <mesh filename="package://robot_description/meshes/merged/unstrander_2_collision.stl"/>
+        <mesh filename="package://qbert_description/meshes/merged/unstrander_2_collision.stl"/>
       </geometry>
     </collision>
@@ -220,5 +220,5 @@
       <origin xyz="-4.50688e-09 -0.000135462 -0.0882216" rpy="1.54515e-14 -0.00433337 -8.26873e-14"/>
       <geometry>
-        <mesh filename="package://robot_description/meshes/merged/compressor_visual.stl"/>
+        <mesh filename="package://qbert_description/meshes/merged/compressor_visual.stl"/>
       </geometry>
       <material name="compressor_parts_material">
@@ -229,5 +229,5 @@
       <origin xyz="-4.50688e-09 -0.000135462 -0.0882216" rpy="1.54515e-14 -0.00433337 -8.26873e-14"/>
       <geometry>
-        <mesh filename="package://robot_description/meshes/merged/compressor_collision.stl"/>
+        <mesh filename="package://qbert_description/meshes/merged/compressor_collision.stl"/>
       </geometry>
     </collision>
@@ -252,5 +252,5 @@
       <origin xyz="-4.50688e-09 -0.000135462 -0.0882216" rpy="3.14159 -1.56646 -3.14159"/>
       <geometry>
-        <mesh filename="package://robot_description/meshes/merged/compressor_2_visual.stl"/>
+        <mesh filename="package://qbert_description/meshes/merged/compressor_2_visual.stl"/>
       </geometry>
       <material name="compressor_2_parts_material">
@@ -261,5 +261,5 @@
       <origin xyz="-4.50688e-09 -0.000135462 -0.0882216" rpy="3.14159 -1.56646 -3.14159"/>
       <geometry>
-        <mesh filename="package://robot_description/meshes/merged/compressor_2_collision.stl"/>
+        <mesh filename="package://qbert_description/meshes/merged/compressor_2_collision.stl"/>
       </geometry>
     </collision>
@@ -284,5 +284,5 @@
       <origin xyz="-4.50688e-09 -0.000135462 -0.0882216" rpy="6.09046e-13 1.56646 -3.14159"/>
       <geometry>
-        <mesh filename="package://robot_description/meshes/merged/compressor_3_visual.stl"/>
+        <mesh filename="package://qbert_description/meshes/merged/compressor_3_visual.stl"/>
       </geometry>
       <material name="compressor_3_parts_material">
@@ -293,5 +293,5 @@
       <origin xyz="-4.50688e-09 -0.000135462 -0.0882216" rpy="6.09046e-13 1.56646 -3.14159"/>
       <geometry>
-        <mesh filename="package://robot_description/meshes/merged/compressor_3_collision.stl"/>
+        <mesh filename="package://qbert_description/meshes/merged/compressor_3_collision.stl"/>
       </geometry>
     </collision>
@@ -317,5 +317,5 @@
       <origin xyz="-4.50688e-09 -0.000135462 -0.0882216" rpy="-3.14159 0.00433337 7.49258e-14"/>
       <geometry>
-        <mesh filename="package://robot_description/meshes/merged/compressor_4_visual.stl"/>
+        <mesh filename="package://qbert_description/meshes/merged/compressor_4_visual.stl"/>
       </geometry>
       <material name="compressor_4_parts_material">
@@ -326,5 +326,5 @@
       <origin xyz="-4.50688e-09 -0.000135462 -0.0882216" rpy="-3.14159 0.00433337 7.49258e-14"/>
       <geometry>
-        <mesh filename="package://robot_description/meshes/merged/compressor_4_collision.stl"/>
+        <mesh filename="package://qbert_description/meshes/merged/compressor_4_collision.stl"/>
       </geometry>
     </collision>
@@ -358,5 +358,5 @@
       <origin xyz="3.37134e-09 -8.22904e-05 -0.0767445" rpy="-3.14159 -7.46793e-14 -3.14159"/>
       <geometry>
-        <mesh filename="package://robot_description/meshes/merged/solid_gripper_visual.stl"/>
+        <mesh filename="package://qbert_description/meshes/merged/solid_gripper_visual.stl"/>
       </geometry>
       <material name="solid_gripper_parts_material">
@@ -367,5 +367,5 @@
       <origin xyz="3.37134e-09 -8.22904e-05 -0.0767445" rpy="-3.14159 -7.46793e-14 -3.14159"/>
       <geometry>
-        <mesh filename="package://robot_description/meshes/merged/solid_gripper_collision.stl"/>
+        <mesh filename="package://qbert_description/meshes/merged/solid_gripper_collision.stl"/>
       </geometry>
     </collision>
@@ -390,5 +390,5 @@
       <origin xyz="3.37134e-09 -8.22904e-05 -0.0767445" rpy="-3.25851e-15 -1.5708 0"/>
       <geometry>
-        <mesh filename="package://robot_description/meshes/merged/solid_gripper_2_visual.stl"/>
+        <mesh filename="package://qbert_description/meshes/merged/solid_gripper_2_visual.stl"/>
       </geometry>
       <material name="solid_gripper_2_parts_material">
@@ -399,5 +399,5 @@
       <origin xyz="3.37134e-09 -8.22904e-05 -0.0767445" rpy="-3.25851e-15 -1.5708 0"/>
       <geometry>
-        <mesh filename="package://robot_description/meshes/merged/solid_gripper_2_collision.stl"/>
+        <mesh filename="package://qbert_description/meshes/merged/solid_gripper_2_collision.stl"/>
       </geometry>
     </collision>
@@ -423,5 +423,5 @@
       <origin xyz="3.37134e-09 -8.22904e-05 -0.0767445" rpy="-3.14159 1.5708 0"/>
       <geometry>
-        <mesh filename="package://robot_description/meshes/merged/solid_gripper_3_visual.stl"/>
+        <mesh filename="package://qbert_description/meshes/merged/solid_gripper_3_visual.stl"/>
       </geometry>
       <material name="solid_gripper_3_parts_material">
@@ -432,5 +432,5 @@
       <origin xyz="3.37134e-09 -8.22904e-05 -0.0767445" rpy="-3.14159 1.5708 0"/>
       <geometry>
-        <mesh filename="package://robot_description/meshes/merged/solid_gripper_3_collision.stl"/>
+        <mesh filename="package://qbert_description/meshes/merged/solid_gripper_3_collision.stl"/>
       </geometry>
     </collision>
@@ -456,5 +456,5 @@
       <origin xyz="3.37134e-09 -8.22904e-05 -0.0767445" rpy="1.69099e-14 9.1368e-14 3.14159"/>
       <geometry>
-        <mesh filename="package://robot_description/meshes/merged/solid_gripper_4_visual.stl"/>
+        <mesh filename="package://qbert_description/meshes/merged/solid_gripper_4_visual.stl"/>
       </geometry>
       <material name="solid_gripper_4_parts_material">
@@ -465,5 +465,5 @@
       <origin xyz="3.37134e-09 -8.22904e-05 -0.0767445" rpy="1.69099e-14 9.1368e-14 3.14159"/>
       <geometry>
-        <mesh filename="package://robot_description/meshes/merged/solid_gripper_4_collision.stl"/>
+        <mesh filename="package://qbert_description/meshes/merged/solid_gripper_4_collision.stl"/>
       </geometry>
     </collision>
@@ -489,5 +489,5 @@
       <origin xyz="0.000712425 -0.000140815 -0.0757529" rpy="-3.14159 0.785398 5.91473e-14"/>
       <geometry>
-        <mesh filename="package://robot_description/meshes/merged/roller_gripper_visual.stl"/>
+        <mesh filename="package://qbert_description/meshes/merged/roller_gripper_visual.stl"/>
       </geometry>
       <material name="roller_gripper_parts_material">
@@ -498,5 +498,5 @@
       <origin xyz="0.000712425 -0.000140815 -0.0757529" rpy="-3.14159 0.785398 5.91473e-14"/>
       <geometry>
-        <mesh filename="package://robot_description/meshes/merged/roller_gripper_collision.stl"/>
+        <mesh filename="package://qbert_description/meshes/merged/roller_gripper_collision.stl"/>
       </geometry>
     </collision>
@@ -521,5 +521,5 @@
       <origin xyz="0.000712425 -0.000140815 -0.0757529" rpy="3.14159 -0.785398 5.35124e-14"/>
       <geometry>
-        <mesh filename="package://robot_description/meshes/merged/roller_gripper_2_visual.stl"/>
+        <mesh filename="package://qbert_description/meshes/merged/roller_gripper_2_visual.stl"/>
       </geometry>
       <material name="roller_gripper_2_parts_material">
@@ -530,5 +530,5 @@
       <origin xyz="0.000712425 -0.000140815 -0.0757529" rpy="3.14159 -0.785398 5.35124e-14"/>
       <geometry>
-        <mesh filename="package://robot_description/meshes/merged/roller_gripper_2_collision.stl"/>
+        <mesh filename="package://qbert_description/meshes/merged/roller_gripper_2_collision.stl"/>
       </geometry>
     </collision>
@@ -554,5 +554,5 @@
       <origin xyz="0.000712425 -0.000140815 -0.0757529" rpy="5.07794e-14 -0.785398 -5.6309e-14"/>
       <geometry>
-        <mesh filename="package://robot_description/meshes/merged/roller_gripper_3_visual.stl"/>
+        <mesh filename="package://qbert_description/meshes/merged/roller_gripper_3_visual.stl"/>
       </geometry>
       <material name="roller_gripper_3_parts_material">
@@ -563,5 +563,5 @@
       <origin xyz="0.000712425 -0.000140815 -0.0757529" rpy="5.07794e-14 -0.785398 -5.6309e-14"/>
       <geometry>
-        <mesh filename="package://robot_description/meshes/merged/roller_gripper_3_collision.stl"/>
+        <mesh filename="package://qbert_description/meshes/merged/roller_gripper_3_collision.stl"/>
       </geometry>
     </collision>
@@ -587,5 +587,5 @@
       <origin xyz="0.000712425 -0.000140815 -0.0757529" rpy="-2.16831e-14 0.785398 -5.58778e-14"/>
       <geometry>
-        <mesh filename="package://robot_description/meshes/merged/roller_gripper_4_visual.stl"/>
+        <mesh filename="package://qbert_description/meshes/merged/roller_gripper_4_visual.stl"/>
       </geometry>
       <material name="roller_gripper_4_parts_material">
@@ -596,5 +596,5 @@
       <origin xyz="0.000712425 -0.000140815 -0.0757529" rpy="-2.16831e-14 0.785398 -5.58778e-14"/>
       <geometry>
-        <mesh filename="package://robot_description/meshes/merged/roller_gripper_4_collision.stl"/>
+        <mesh filename="package://qbert_description/meshes/merged/roller_gripper_4_collision.stl"/>
       </geometry>
     </collision>

Commit message: back to not working

File: src/qbert_description/urdf/qbert.xacro (robot description, xacro)
@@ -44,5 +44,5 @@
     <gazebo>
         <plugin filename="libgz_ros2_control-system.so" name="gz_ros2_control::GazeboSimROS2ControlPlugin">
-            <parameters>$(find qbert_description)/config/qbert_controllers.yaml</parameters>
+            <parameters>$(find qbert_control)/config/qbert_controllers.yaml</parameters>
             <controller_manager_prefix_node_name>controller_manager</controller_manager_prefix_node_name>
         </plugin>

File: src/qbert_description/urdf/qbert_base.xacro (robot description, xacro)
@@ -304,5 +304,4 @@
     <axis xyz="0 0 1"/>
     <limit effort="10" velocity="10" lower="-0.04" upper="0"/>
-    <mimic joint="J3_B_compressor_2" multiplier="1.0"/>
   </joint>
   <!-- Link compressor_4 -->
@@ -337,5 +336,4 @@
     <axis xyz="0 0 1"/>
     <limit effort="10" velocity="10" lower="-0.04" upper="0.0"/>
-    <mimic joint="J3_B_compressor_1" multiplier="1.0"/>
   </joint>
   <!-- Joint from stator to rot_disc -->
@@ -410,5 +408,4 @@
     <axis xyz="0 0 1"/>
     <limit effort="10" velocity="10" lower="-0.04" upper="-6.38378e-16"/>
-    <mimic joint="J2_B_solid_gripper_1" multiplier="1.0"/>
   </joint>
   <!-- Link solid_gripper_3 -->
@@ -443,5 +440,4 @@
     <axis xyz="0 0 1"/>
     <limit effort="10" velocity="10" lower="-0.04" upper="-3.88578e-16"/>
-    <mimic joint="J2_B_solid_gripper_1" multiplier="1.0"/>
   </joint>
   <!-- Link solid_gripper_4 -->
@@ -476,5 +472,4 @@
     <axis xyz="0 0 1"/>
     <limit effort="10" velocity="10" lower="-0.04" upper="-4.44089e-16"/>
-    <mimic joint="J2_B_solid_gripper_1" multiplier="1.0"/>
   </joint>
   <!-- Link roller_gripper -->
@@ -541,5 +536,4 @@
     <axis xyz="0 0 1"/>
     <limit effort="10" velocity="10" lower="-0.04" upper="1.15426e-14"/>
-    <mimic joint="J2_C_roller_gripper_1" multiplier="1.0"/>
   </joint>
   <!-- Link roller_gripper_3 -->
@@ -574,5 +568,4 @@
     <axis xyz="0 0 1"/>
     <limit effort="10" velocity="10" lower="-0.04" upper="1.16236e-14"/>
-    <mimic joint="J2_C_roller_gripper_1" multiplier="1.0"/>
   </joint>
   <!-- Link roller_gripper_4 -->
@@ -607,5 +600,4 @@
     <axis xyz="0 0 1"/>
     <limit effort="10" velocity="10" lower="-0.04" upper="1.14617e-14"/>
-    <mimic joint="J2_C_roller_gripper_1" multiplier="1.0"/>
   </joint>
   <!-- Joint from linear_gantry__configuration_festo to stator -->

File: src/qbert_description/urdf/qbert_ros2control.xacro (robot description, xacro)
@@ -1,15 +1,84 @@
 <?xml version="1.0"?>
 <robot name="qbert">
-    <ros2_control name="qbert" type="system">
-        <hardware>
-            <plugin>gz_ros2_control/GazeboSimSystem</plugin>
-        </hardware>
-        <joint name="J2_A_rotor">
-            <command_interface name="position">
-                <param name="min">-3.1415</param>
-                <param name="max">3.1415</param>
-            </command_interface>
-            <state_interface name="position"/>
-        </joint>
-    </ros2_control>
+  <ros2_control name="qbert" type="system">
+    <hardware>
+      <plugin>gz_ros2_control/GazeboSimSystem</plugin>
+    </hardware>
+    <!-- Linear Gantry -->
+    <joint name="J1_gantry">
+      <command_interface name="position"/>
+      <state_interface name="position"/>
+      <limit lower="-0.27" upper="0.27" effort="10" velocity="10"/>
+    </joint>
+    <!-- Unstrander -->
+    <joint name="J4_unstrander">
+      <command_interface name="position"/>
+      <state_interface name="position"/>
+      <limit lower="-0.04" upper="0.0" effort="10" velocity="10"/>
+    </joint>
+    <!-- Tool Disc + Rotor -->
+    <joint name="joint_J3_A_tool_disc">
+      <command_interface name="position"/>
+      <state_interface name="position"/>
+      <limit lower="-0.2" upper="0.0" effort="10" velocity="10"/>
+    </joint>
+    <joint name="J2_A_rotor">
+      <command_interface name="position"/>
+      <state_interface name="position"/>
+      <limit lower="-3.14593" upper="3.13726" effort="10" velocity="10"/>
+    </joint>
+    <!-- Compressor -->
+    <joint name="J3_B_compressor_1">
+      <command_interface name="position"/>
+      <state_interface name="position"/>
+      <limit lower="-0.04" upper="0.0" effort="10" velocity="10"/>
+    </joint>
+    <joint name="J3_B_compressor_2">
+      <command_interface name="position"/>
+      <state_interface name="position"/>
+      <limit lower="-0.04" upper="0.0" effort="10" velocity="10"/>
+    </joint>
+    <joint name="J3_B_compressor_3">
+      <command_interface name="position"/>
+      <state_interface name="position"/>
+      <limit lower="-0.04" upper="0.0" effort="10" velocity="10"/>
+    </joint>
+    <joint name="J3_B_compressor_4">
+      <command_interface name="position"/>
+      <state_interface name="position"/>
+      <limit lower="-0.04" upper="0.0" effort="10" velocity="10"/>
+    </joint>
+    <!-- Gripper -->
+    <joint name="J2_B_solid_gripper_1">
+      <command_interface name="position"/>
+      <state_interface name="position"/>
+      <limit lower="-0.04" upper="0.0" effort="10" velocity="10"/>
+    </joint>
+    <joint name="J2_B_solid_gripper_2">
+      <command_interface name="position"/>
+      <state_interface name="position"/>
+      <limit lower="-0.04" upper="-6.38378e-16" effort="10" velocity="10"/>
+    </joint>
+    <joint name="J2_B_solid_gripper_3">
+      <command_interface name="position"/>
+      <state_interface name="position"/>
+      <limit lower="-0.04" upper="-3.88578e-16" effort="10" velocity="10"/>
+    </joint>
+    <joint name="J2_B_solid_gripper_4">
+      <command_interface name="position"/>
+      <state_interface name="position"/>
+      <limit lower="-0.04" upper="-4.44089e-16" effort="10" velocity="10"/>
+    </joint>
+    <!-- Roller -->
+    <joint name="J2_C_roller_gripper_1">
+      <command_interface name="position"/>
+      <state_interface name="position"/>
+      <limit lower="-0.04" upper="1.15402e-14" effort="10" velocity="10"/>
+    </joint>
+    <joint name="J2_C_roller_gripper_2">
+      <command_interface name="position"/>
+      <state_interface name="position"/>
+      <limit lower="-0.04" upper="1.15426e-14" effort="10" velocity="10"/>
+    </joint>
+  </ros2_control>
 </robot>
