Commit message: added 2 missing grippers

File: src/qbert_description/urdf/qbert_ros2control.xacro (robot description, xacro)
@@ -81,4 +81,14 @@
       <limit lower="-0.04" upper="1.15426e-14" effort="10" velocity="10"/>
     </joint>
+    <joint name="J2_C_roller_gripper_3">
+      <command_interface name="position"/>
+      <state_interface name="position"/>
+      <limit lower="-0.04" upper="1.15402e-14" effort="10" velocity="10"/>
+    </joint>
+    <joint name="J2_C_roller_gripper_4">
+      <command_interface name="position"/>
+      <state_interface name="position"/>
+      <limit lower="-0.04" upper="1.15426e-14" effort="10" velocity="10"/>
+    </joint>
   </ros2_control>
 </robot>
